File: kicad/27C160_Adapter.sch (KiCad schematic (older format))
At the start: 10 parts, among them Q1 BC327, SW1 MS22D16, SW2 DIP, U1 27C4002

Commit message: Shrunk PCB size Converted resistors and transistor to SMD Introduced GND fills Converted to Kicad 5.x
Parts:
- Q1: value BC327 -> BC807; footprint 27C160_Adapter:TO92-EBC -> Package_TO_SOT_SMD:SOT-23; symbol BC327 -> Transistor_BJT:BC807
- R1, R2, R3, R4, R5: footprint 27C160_Adapter:0207_10 -> Resistor_SMD:R_0805_2012Metric; symbol R-EU_0207_10 -> 27C160_Adapter:R-EU_0207_10
- SW1: footprint 27C160_Adapter:MS22D16 -> Button_Switch_THT:SW_NKK_GW12LJP; symbol MS22D16 -> 27C160_Adapter:MS22D16
- SW2: footprint 27C160_Adapter:EDG-03 -> Button_Switch_THT:SW_DIP_SPSTx03_Slide_9.78x9.8mm_W7.62mm_P2.54mm; symbol SW_DIP-3 -> 27C160_Adapter:SW_DIP-3
- U1: footprint 27C160_Adapter:27C4002 -> Package_DIP:DIP-40_W15.24mm_LongPads; symbol 27C4002 -> 27C160_Adapter:27C4002
- ZX1: symbol 3M_248-3345 -> 27C160_Adapter:3M_248-3345
Connections:
- wire segments 119 -> 130
